File: pcb/pcb/pcb.kicad_pcb (KiCad board)
At the start: 4 copper layers, 75 x 50 mm, 62 parts, among them J1 Conn_01x04_Pin, J2 DE15_Receptacle_HighDensity_M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, J3 MicroSD_Receptacle, J4 AudioJack4, J5 USB_C_Receptacle_PowerOnly_6P, J6 USB_A, J7 USB_A, Q1 Si2300DS, Q2 Si2300DS, Q3 Si2300DS, SW1 SW_Push, SW2 SW_Push, U1 CH32X035G8R6, U2 SRV05-4, U3 CD4066BM, U4 TL072CDR

Commit message: update schematic and pcb
Parts:
- removed C12, C13: 33p, Capacitor_SMD:C_1206_3216Metric
- removed U3: CD4066BM, Package_SO:SO-14_3.9x8.65mm_P1.27mm
- J4: footprint Connector_Audio:Jack_3.5mm_PJ320D_Horizontal -> Connector_Audio:Jack_3.5mm_PJ320E_Horizontal
- J6: value USB_A -> Conn_01x04_Pin; footprint Connector_USB:USB2_A_Female_Short_14.6x10 -> Connector_PinHeader_2.54mm:PinHeader_1x04_P2.54mm_Vertical
- R19, R20: value 270 -> 270R
- R24: value 330 -> 330R
- R4, R5: value 47 -> 47R
- R6, R7, R8: value 470 -> 470R
- moved J6 19.8 mm to (56.5, 52.8), turned to 90 degrees
- moved D5 15.0 mm to (57.2, 75.5)
- moved C8 14.8 mm to (44.3, 50.5)
- moved R19 14.1 mm to (57.2, 70.2), turned to -90 degrees
- moved J7 14.0 mm to (42.1, 40.0)
- moved R27 12.4 mm to (51.8, 40.9)
- moved R26 12.0 mm to (51.8, 38.6)
- moved D3 11.7 mm to (44.2, 53.8), turned to 180 degrees
- moved J5 10.0 mm to (41.6, 61.8)
- moved C1 6.95 mm to (47.2, 69.8)
- moved R1 6.95 mm to (48.6, 66.0)
- moved SW1 6.95 mm to (45.2, 74.6)
- moved J4 4.39 mm to (108.8, 67.0), turned to 180 degrees
- moved SW2 2.70 mm to (59.2, 35.8)
- moved C7 0.31 mm to (78.7, 36.0)
Connections:
- J2 pad 11: Net-(U1-PB11/T1C3/T2C1N_/RX1) -> Net-(U1-PB10/TX1/T1C2)
- J6 pad 2: Net-(J6-D-) -> GND
- J6 pad 3: Net-(J6-D+) -> Net-(J6-Pin_3)
- J6 pad 4: GND -> Net-(J6-Pin_4)
- R26 pad 2: Net-(C12-Pad1) -> Net-(J7-D-)
- R27 pad 2: Net-(C13-Pad1) -> Net-(J7-D+)
- R5 pad 1: Net-(U1-PB10/TX1/T1C2) -> Net-(U1-PB11/T1C3/T2C1N_/RX1)
- U1 pad 10: Net-(U1-PA1/RTS2/T2C2/C1O/O1N2/O2N2/A1) -> Net-(J6-Pin_3)
- U1 pad 11: Net-(U1-PA2/TX2/T2C3/O2O1/T2ET_/C3N0/A2) -> Net-(J6-Pin_4)
Routing:
- net +5V: track 276.9 -> 224.1 mm, vias 18 -> 15
- net Net-(U1-PA1/RTS2/T2C2/C1O/O1N2/O2N2/A1): track 36.5 -> 0.00 mm, vias 3 -> 0
- net Net-(U1-PA2/TX2/T2C3/O2O1/T2ET_/C3N0/A2): track 34.4 -> 0.00 mm, vias 3 -> 0
- net Net-(J6-Pin_3): track 0.00 -> 21.2 mm
- net Net-(J6-Pin_4): track 0.00 -> 18.2 mm
- net Net-(C13-Pad1): track 18.2 -> 0.00 mm, vias 2 -> 0
- net GND: track 43.6 -> 25.8 mm, vias 74 -> 52
- net Net-(C12-Pad1): track 16.9 -> 0.00 mm
- net Net-(U1-PB11/T1C3/T2C1N_/RX1): track 30.2 -> 13.8 mm, vias 1 -> 0
- net Net-(U1-PB10/TX1/T1C2): track 16.8 -> 32.8 mm
- net Net-(J6-D-): track 13.9 -> 0.00 mm
- net Net-(J6-D+): track 10.4 -> 0.00 mm
- net Net-(U1-PA3/T2C4/O1O0/T3C1_/RX2/A3): track 47.4 -> 54.4 mm
- net Net-(J5-CC2): track 59.3 -> 52.3 mm
- net Net-(D2-K): track 59.9 -> 53.3 mm
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- removed copper zone on In1.Cu, net GND
- removed copper zone on In2.Cu, net GND
Other:
- copper layers 4 -> 2
- board text added: "1"
- board text added: "11"
- board text added: "15"
- board text added: "3.3V"
- board text added: "5"
- board text added: "5V"
- board text added: "D+"
- board text added: "D-"
- board text added: "DBG/I2C_RX"
- board text added: "GND"
- board text added: "I2C_TX"
- board text added: "PA1"
- board text added: "PA2"
- board text added: "RX"
- board text added: "S"
- board text added: "SW1"
- board text added: "SW2"
- board text added: "T"
- board text added: "TX"
- board text added: "USB DATA"
- board text added: "USB PD INPUT 5V"
- board text removed: "PORT_SEL"
- board text removed: "PWR 5V"
- board text removed: "PWR3V"
- board text removed: "USB 1"
- board text removed: "USB 2"
- board text removed: "USB PD"
