File: pcb/pcb/pcb.kicad_sch (KiCad schematic)
At the start: 62 parts, among them J1 Conn_01x04_Pin, J2 DE15_Receptacle_HighDensity_M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, J3 MicroSD_Receptacle, J4 AudioJack4, J5 USB_C_Receptacle_PowerOnly_6P, J6 USB_A, J7 USB_A, Q1 Si2300DS, Q2 Si2300DS, Q3 Si2300DS, SW1 SW_Push, SW2 SW_Push, U1 CH32X035G8R6, U2 SRV05-4, U3 CD4066BM, U4 TL072CDR

Commit message: update schematic and pcb
Parts:
- removed C12, C13: 33p, Capacitor_SMD:C_1206_3216Metric, symbol Device:C
- removed J6: USB_A, Connector_USB:USB2_A_Female_Short_14.6x10, symbol Connector:USB_A
- removed U3: CD4066BM, Package_SO:SO-14_3.9x8.65mm_P1.27mm, symbol Analog_Switch:CD4066BM
- added J6: Conn_01x04_Pin, Connector_PinHeader_2.54mm:PinHeader_1x04_P2.54mm_Vertical, symbol Connector:Conn_01x04_Pin
- J4: footprint Connector_Audio:Jack_3.5mm_PJ320D_Horizontal -> Connector_Audio:Jack_3.5mm_PJ320E_Horizontal
- R19, R20: value 270 -> 270R
- R24: value 330 -> 330R
- R4, R5: value 47 -> 47R
- R6, R7, R8: value 470 -> 470R
Connections:
- net +5V: now also J6.1 (Pin_1)
- net GND: now also J6.2 (Pin_2)
- net at R27.2: now also J7.3 (D+)
- net at J7.2 (D-): now also R26.2
- net at U1.11 (PA2/TX2/T2C3/O2O1/T2ET_/C3N0/A2): now also J6.4 (Pin_4)
- net at J2.11: now also U1.25 (PB10/TX1/T1C2); no longer U1.26 (PB11/T1C3/T2C1N_/RX1)
- net at R5.1: now also U1.26 (PB11/T1C3/T2C1N_/RX1); no longer U1.25 (PB10/TX1/T1C2)
- net at U1.10 (PA1/RTS2/T2C2/C1O/O1N2/O2N2/A1): now also J6.3 (Pin_3)
Other:
- title: CH32X035 -> RVPC2
- moved on the sheet: C1, C2, C8, D3, J5, J7, R1, R2, R26, R27, SW1, SW2
